Commit message: Reduce weight of VLP16 sensor

File: velodyne_description/urdf/VLP-16.urdf.xacro (robot description, xacro)
@@ -10,5 +10,5 @@
     <link name="${name}_base_link">
       <inertial>
-        <mass value="0.83"/>
+        <mass value="0.01"/>
         <origin xyz="0 0 0.03585"/>
         <inertia ixx="${(0.83 * (3.0*0.0516*0.0516 + 0.0717*0.0717)) / 12.0}" ixy="0" ixz="0"
